Commit message: Make urdf work on dora

File: reachy.urdf (robot description, URDF)
Before this commit: robot reachy, 31 links, 30 joints
Links:
- link bottom_orbita_arm: geometry collision cylinder length=0.0 radius=0.0; visual mesh filename=meshes/orbita_arm.dae
- link head: geometry collision cylinder length=0.15 radius=0.06; visual mesh filename=meshes/head.dae
- link l_antenna: geometry collision cylinder length=0.0 radius=0.0; visual mesh filename=meshes/antenna.dae
- link l_forearm: geometry collision cylinder length=0.09 radius=0.04; visual mesh filename=meshes/forearm.dae
- link l_gripper_finger: geometry collision box size=0.1 0.012 0.035; visual mesh filename=meshes/l_gripper_finger.dae
- link l_gripper_thumb: geometry collision box size=0.1 0.012 0.035; visual mesh filename=meshes/l_gripper_thumb.dae
- link l_shoulder: geometry collision cylinder length=0.09 radius=0.035; visual mesh filename=meshes/shoulder.dae
- link l_shoulder_x: geometry collision cylinder length=0.04 radius=0.035; visual mesh filename=meshes/shoulder_x.dae
- link l_upper_arm: geometry collision cylinder length=0.25 radius=0.04; visual mesh filename=meshes/upper_arm.dae
- link l_wrist: geometry collision cylinder length=0.14 radius=0.035; visual mesh filename=meshes/wrist.dae
- link l_wrist2hand: geometry collision cylinder length=0.06 radius=0.03; visual mesh filename=meshes/wrist2hand.dae
- link middle_orbita_arm: geometry collision cylinder length=0.0 radius=0.0; visual mesh filename=meshes/orbita_arm.dae
- link r_antenna: geometry collision cylinder length=0.0 radius=0.0; visual mesh filename=meshes/antenna.dae
- link r_forearm: geometry collision cylinder length=0.09 radius=0.04; visual mesh filename=meshes/forearm.dae
- link r_gripper_finger: geometry collision box size=0.1 0.012 0.035; visual mesh filename=meshes/r_gripper_finger.dae
- link r_gripper_thumb: geometry collision box size=0.1 0.012 0.035; visual mesh filename=meshes/r_gripper_thumb.dae
- link r_shoulder: geometry collision cylinder length=0.09 radius=0.035; visual mesh filename=meshes/shoulder.dae
- link r_shoulder_x: geometry collision cylinder length=0.04 radius=0.035; visual mesh filename=meshes/shoulder_x.dae
- link r_upper_arm: geometry collision cylinder length=0.25 radius=0.04; visual mesh filename=meshes/upper_arm.dae
- link r_wrist: geometry collision cylinder length=0.14 radius=0.035; visual mesh filename=meshes/wrist.dae
- link r_wrist2hand: geometry collision cylinder length=0.06 radius=0.03; visual mesh filename=meshes/wrist2hand.dae
- link top_orbita_arm: geometry collision cylinder length=0.0 radius=0.0; visual mesh filename=meshes/orbita_arm.dae
- link torso: geometry collision box size=0.11 0.2 0.32; visual mesh filename=meshes/torso.dae
